File: Minima DG/untitled.brd (EAGLE design)
At the start: 100 x 80 mm, 33 parts, among them IC1 MEGA8-P, IC3 7805, Q1 16MHz, X2 VFO

Commit message: Added BOM files, remove unneeded files.
Parts:
- moved C4 30.5 mm to (9.84, 36.8)
- moved C7 30.5 mm to (85.1, 42.5)
- moved C8 30.5 mm to (76.8, 42.5)
- moved IC4 30.5 mm to (81.0, 34.9)
- moved Q1 30.5 mm to (46.7, 14.0)
- moved R4 30.5 mm to (76.5, 9.53)
- moved C2 30.5 mm to (44.1, 10.2)
- moved C3 30.5 mm to (49.2, 10.2)
- moved DIS1 30.5 mm to (56.8, 28.6)
- moved IC1 30.5 mm to (42.9, 23.5)
- moved IC2 30.5 mm to (11.1, 20.6)
- moved 12V 30.5 mm to (89.9, 4.45)
- moved 5V 30.5 mm to (21.3, 4.45)
- moved BAND 30.5 mm to (50.5, 4.45)
- moved BFO 30.5 mm to (39.1, 4.45)
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Routing:
- added copper zone on layer 1, net GND
Other:
- board size 100 x 80 mm -> 100 x 48.2 mm
