File: Minima MB/untitled.sch (EAGLE design)
At the start: 204 parts, among them IC1 78L05, K1 G5V1, K2 G5V-2, K3 G5V1, K4 G5V1, Q10 2N3904, Q11 2N3904, Q12 2N3904, Q13 2N3904, Q14 2N3904, Q15 2N3904, Q16 2N3904, Q17 BFO, Q18 J310, Q19 J310, Q20 2N3904, Q21 2N3906, Q22 2N3904, Q23 2N3904, Q24 2N3904, Q25 2N3904, Q26 2N3904, Q27 2N3904, Q28 2N3904, Q29 2N3904, Q30 2N3904, Q39 2N3904, Q8 2N3904, X1 VFO, X3 PA

Commit message: Added BOM files, remove unneeded files.
Parts:
- C50: value (none) -> 1 uF
- C57, C68, C69: value (none) -> 22 pF
- R14: value (none) -> 10k
- R48: value 10u -> 10
Other:
- moved on the sheet: C23, C42, C56, C57, C58, C59, C60, C61, C62, C63, C64, C65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
